Commit message: update

File: examples/vx300s.urdf (robot description, URDF)
Before this commit: robot vx300s, 14 links, 13 joints
Links:
- removed link /left_finger_link
- removed link /right_finger_link
Joints:
- removed joint left_finger
- removed joint right_finger

Commit message: update need to change everything to ee_gripper_frame

File: examples/vx300s.urdf (robot description, URDF)
Before this commit: robot vx300s, 12 links, 11 joints
Links:
- removed link /ee_gripper_link
- removed link /fingers_link
- removed link /gripper_bar_link
Joints:
- removed joint ee_bar
- removed joint ee_gripper
- removed joint gripper_bar
- joint elbow: origin xyz=0.05955 0 0.3 rpy=3.141592653589793 0 0 -> xyz=0.05955 0 0.3 rpy=0 0 0
- joint gripper: origin xyz=0.005675 0 0 rpy=0 0 0 -> xyz=0 0 0 rpy=0 0 0
- joint waist: origin xyz=0 0 0.0787 rpy=0 0 0 -> xyz=0 0 0.079 rpy=0 0 0
- joint wrist_rotate: origin xyz=0.069744 0 0 rpy=-3.141592653589793 0 0 -> xyz=0.069744 0 0 rpy=0 0 0

Commit message: align to ee_gripper_link

File: examples/vx300s.urdf (robot description, URDF)
Before this commit: robot vx300s, 9 links, 8 joints
Joints:
- joint gripper: origin xyz=0 0 0 rpy=0 0 0 -> xyz=0.064 0 0 rpy=0 0 0
