Commit message: update

File: examples/spot_description/spot_arm.urdf (robot description, URDF)
Before this commit: robot spot_arm, 9 links, 8 joints
Links:
- removed link payload_link
- link arm_link_fngr: geometry collision box size=0.05 0.2 0.1; collision mesh filename=/home/jiahe/pinocchio/examples/spot_description/meshes/arm/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
Joints:
- removed joint payload_fix
